File: hardware/vco1/vco1.kicad_pcb (KiCad board)
At the start: 2 copper layers, 50 x 100 mm, 77 parts, among them J1 AudioJack2_SwitchT, J10 Conn_01x02_Pin, J2 AudioJack2_SwitchT, J3 AudioJack2_SwitchT, J4 AudioJack2_SwitchT, J5 Conn_02x08_Odd_Even, J6 AudioJack2_SwitchT, J7 AudioJack2_SwitchT, J8 Conn_01x02_Pin, J9 Conn_01x02_Pin, Q1 2N3904, Q2 2N3906, U1 40106, U2 TL074, U3 TL074

Commit message: added PDF of schematic & board rendering
Other:
- board text added: "JLCJLCJLCJLC"
Changed lines of the file:
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@@
 		(allow_soldermask_bridges_in_footprints no)
 		(pcbplotparams
-			(layerselection 0x00010fc_ffffffff)
+			(layerselection 0x0001330_ffffffff)
 			(plot_on_all_layers_selection 0x0000000_00000000)
 			(disableapertmacros no)
@@
 			(sketchpadsonfab no)
 			(subtractmaskfromsilk no)
-			(outputformat 1)
+			(outputformat 4)
 			(mirror no)
-			(drillshape 1)
+			(drillshape 0)
 			(scaleselection 1)
-			(outputdirectory "")
+			(outputdirectory "/home/dmcguire/Source/eurorack/vco-1/docs/")
 		)
 	)
@@
 		(tags "CP Radial series Radial pin pitch 2.50mm  diameter 5mm Electrolytic Capacitor")
 		(property "Reference" "C9"
-			(at 4.253113 2.032 360)
+			(at 4.253113 2.032 0)
 			(layer "F.SilkS")
 			(effects
@@
 		)
 		(property "Value" "47u"
-			(at 1.25 3.75 360)
+			(at 1.25 3.75 0)
 			(layer "F.Fab")
 			(effects
@@
 		)
 		(fp_text user "${REFERENCE}"
-			(at 1.25 0 360)
+			(at 1.25 0 0)
 			(layer "F.Fab")
 			(effects
@@
 		(tags "CP Radial series Radial pin pitch 2.50mm  diameter 5mm Electrolytic Capacitor")
 		(property "Reference" "C8"
-			(at -1.524 -2.5 360)
+			(at -1.524 -2.5 0)
 			(layer "F.SilkS")
 			(effects
@@
 		)
 		(property "Value" "47u"
-			(at 1.25 3.75 360)
+			(at 1.25 3.75 0)
 			(layer "F.Fab")
 			(effects
@@
 		)
 		(fp_text user "${REFERENCE}"
-			(at 1.25 0 360)
+			(at 1.25 0 0)
 			(layer "F.Fab")
 			(effects
@@
 		(tags "Resistor Axial_DIN0204 series Axial Vertical pin pitch 2.54mm 0.167W length 3.6mm diameter 1.6mm")
 		(property "Reference" "R27"
-			(at 5.284 0 360)
+			(at 5.284 0 0)
 			(layer "F.SilkS")
 			(effects
@@
 		)
 		(property "Value" "100k"
-			(at 1.27 1.92 360)
+			(at 1.27 1.92 0)
 			(layer "F.Fab")
 			(effects
@@
 		)
 		(fp_text user "${REFERENCE}"
-			(at 1.27 -1.92 360)
+			(at 1.27 -1.92 0)
 			(layer "F.Fab")
 			(effects
@@
 		(layer "Edge.Cuts")
 	)
+	(gr_text "JLCJLCJLCJLC"
+		(at 183.642 109.728 0)
+		(layer "B.SilkS")
+		(effects
+			(font
+				(size 1 1)
+				(thickness 0.15)
+			)
+			(justify left bottom mirror)
+		)
+	)
 	(gr_text "PWM CV"
